File: Schematics/PicoBalloon/PicoBalloon.kicad_pcb (KiCad board)
At the start: 4 copper layers, 26 x 50 mm, 48 parts, among them J1 SOLAR_R, J2 SOLAR_L, J3 LORA_ANT, J4 SWD, U1 ATGM336H, U2 AT2659S, U3 TMP235A4DCKR, U4 STM32F103C8Tx, U5 MCP1640Bx-xCHY, U6 MT9700

Commit message: Added gerber files for v1.0
Routing:
- net GND: vias 65 -> 87
- net /V_SUPERCAP_SENSE: vias 2 -> 3

Commit message: Started working on PCB A1.1
Parts:
- removed kibuzzard-688BBE2B: G***, kibuzzard-688BBE2B
- added kibuzzard-68A4CDDF: G***, kibuzzard-68A4CDDF, F.Cu at (161.0, 97.2)
- moved C2 6.39 mm to (149.4, 89.5)
- moved D1 1.76 mm to (159.3, 105.3)
- moved D2 1.76 mm to (159.3, 103.6)
- moved R3 1.76 mm to (156.0, 105.3)
- moved R4 1.76 mm to (156.0, 103.6)
- moved J4 0.70 mm to (158.5, 101.0)
- moved J3 0.61 mm to (161.3, 124.7)
- moved C4 0.56 mm to (161.0, 114.1)
- moved C3 0.49 mm to (160.5, 117.7)
- moved U2 0.20 mm to (150.3, 92.1), turned to 180 degrees
Connections:
- L1 pad 1: Net-(U2-RF_OUT) -> Net-(U2-RF_IN)
- U2 pad 1: Net-(U1-RF_IN) -> Net-(U2-RF_IN)
- U2 pad 4: Net-(U2-RF_OUT) -> Net-(U1-RF_IN)
Routing:
- net GND: track 77.5 -> 63.3 mm, vias 87 -> 83
- net +3V3: track 189.3 -> 180.3 mm, vias 5 -> 7
- net Net-(U2-RF_IN): track 0.00 -> 2.56 mm
- net Net-(U2-RF_OUT): track 2.45 -> 0.00 mm
- net Net-(U4-PB14): track 4.88 -> 3.57 mm
- net /LORA_SCK: track 22.1 -> 21.1 mm
- net /SUPERCAP_EN: track 35.8 -> 34.8 mm
- net /LORA_CS: track 24.0 -> 23.1 mm
- net /SWDIO: track 5.22 -> 4.48 mm
- net Net-(U4-PB13): track 6.16 -> 5.51 mm
- net Net-(J3-Pin_1): track 3.94 -> 3.32 mm
- net /LORA_RST: track 21.4 -> 21.9 mm
- net /V_SUPERCAP_SENSE: vias 3 -> 2
Other:
- board size 26 x 50 mm -> 24 x 50 mm
- board text removed: "Pícaro V1.0 Contact @LabGluon if found! Safe device Scientific project."
