File: Schematics/PicoBalloon/PicoBalloon.kicad_pcb (KiCad board)
At the start: 4 copper layers, 24 x 50 mm, 48 parts, among them J1 SOLAR_R, J2 SOLAR_L, J3 LORA_ANT, J4 SWD, U1 ATGM336H, U2 AT2659S, U3 TMP235A4DCKR, U4 STM32F103C8Tx, U5 MCP1640Bx-xCHY, U6 MT9700

Commit message: Version PCB A1.1
Parts:
- added R12: 33, Resistor_SMD:R_0603_1608Metric_Pad0.98x0.95mm_HandSolder, B.Cu at (142.0, 97.8)
- added R13: 0R, Resistor_SMD:R_0603_1608Metric_Pad0.98x0.95mm_HandSolder, B.Cu at (144.2, 103.9)
- added R14: 0R, Resistor_SMD:R_0603_1608Metric_Pad0.98x0.95mm_HandSolder, B.Cu at (145.0, 97.8)
- added U7: MT9700, Package_TO_SOT_SMD:SOT-23-5_HandSoldering, B.Cu at (143.5, 101.3)
- C15: value 10F -> 15F
- R10: value 33 -> 16.5
- R3, R4: value 1k -> 3k3
Connections:
- C1 pad 2: +3V3 -> Net-(U1-VBAT)
- C2 pad 2: +3V3 -> Net-(U2-VDD)
- U1 pad 6: +3V3 -> Net-(U1-VBAT)
- U1 pad 8: +3V3 -> Net-(U1-VBAT)
- U2 pad 6: +3V3 -> Net-(U2-VDD)
- U4 pad 13: unconnected-(U4-PA3-Pad13) -> /GPS_SUPPLY_ENABLE
Routing:
- net +3V3: track 180.3 -> 152.5 mm
- net Net-(U1-VBAT): track 0.00 -> 12.2 mm
- net Net-(U2-VDD): track 0.00 -> 9.66 mm
- net /SUPPLY_GPS_LNA: track 0.00 -> 7.34 mm
- net /GPS_SUPPLY_ENABLE: track 0.00 -> 6.15 mm, vias 0 -> 1
- net Net-(U7-Set): track 0.00 -> 1.69 mm
- net /V_SUPERCAP_SENSE: track 35.6 -> 37.2 mm
- net /SUPERCAP_EN: track 34.8 -> 36.1 mm
- net /V_SOLAR: track 19.6 -> 20.8 mm
- net /LORA_SCK: track 21.1 -> 22.0 mm
- net GND: track 63.3 -> 62.4 mm, vias 83 -> 93
- net /LORA_CS: track 23.1 -> 23.9 mm
