File: Schematics/PicoBalloon/power.kicad_sch (KiCad schematic)
At the start: 11 parts, among them U2 MCP1640Bx-xCHY, U6 MT9700

Commit message: Updated R10 size and datasheets
Parts:
- C15: renamed from C2; footprint (none) -> Package_TO_SOT_SMD:SOT-23-6_Handsoldering
- R10: renamed from R7; footprint Resistor_SMD:R_0603_1608Metric_Pad0.98x0.95mm_HandSolder -> Resistor_SMD:R_2010_5025Metric_Pad1.40x2.65mm_HandSolder; LCSC (none) -> https://lcsc.com/product-detail/image/FRC2010J330-TS_C29075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
- U5: renamed from U2; LCSC (none) -> https://lcsc.com/product-detail/DC-DC-Converters_MICROCHIP-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
- renumbered C1 to C13, C3 to C14, L1 to L2, R8 to R11, R11 to R7, R1 to R8, R2 to R9
Changed lines of the file:
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@@
 		(on_board yes)
 		(dnp no)
-		(property "Reference" "#PWR02"
+		(property "Reference" "#PWR027"
 			(at 139.7 95.25 0)
 			(effects
@@
 			(project "PicoBalloon"
 				(path "/0b983980-f4cd-49d3-aecb-9bdb75de805b/ab4eed9b-d1e6-4c70-aac7-9c30168f7593"
-					(reference "#PWR02")
+					(reference "#PWR027")
 					(unit 1)
 				)
@@
 		(on_board yes)
 		(dnp no)
-		(property "Reference" "R8"
+		(property "Reference" "R11"
 			(at 168.656 82.804 0)
 			(effects
@@
 			(project "PicoBalloon"
 				(path "/0b983980-f4cd-49d3-aecb-9bdb75de805b/ab4eed9b-d1e6-4c70-aac7-9c30168f7593"
-					(reference "R8")
+					(reference "R11")
 					(unit 1)
 				)
@@
 		(on_board yes)
 		(dnp no)
-		(property "Reference" "#PWR011"
+		(property "Reference" "#PWR030"
 			(at 181.61 95.25 0)
 			(effects
@@
 			(project "PicoBalloon"
 				(path "/0b983980-f4cd-49d3-aecb-9bdb75de805b/ab4eed9b-d1e6-4c70-aac7-9c30168f7593"
-					(reference "#PWR011")
+					(reference "#PWR030")
 					(unit 1)
 				)
@@
 		(on_board yes)
 		(dnp no)
-		(property "Reference" "#PWR030"
+		(property "Reference" "#PWR028"
 			(at 149.86 88.9 0)
 			(effects
@@
 			(project "PicoBalloon"
 				(path "/0b983980-f4cd-49d3-aecb-9bdb75de805b/ab4eed9b-d1e6-4c70-aac7-9c30168f7593"
-					(reference "#PWR030")
+					(reference "#PWR028")
 					(unit 1)
 				)
@@
 		(dnp no)
 		(fields_autoplaced yes)
-		(property "Reference" "C3"
+		(property "Reference" "C14"
 			(at 152.4 77.4762 0)
 			(effects
@@
 			(project "PicoBalloon"
 				(path "/0b983980-f4cd-49d3-aecb-9bdb75de805b/ab4eed9b-d1e6-4c70-aac7-9c30168f7593"
-					(reference "C3")
+					(reference "C14")
 					(unit 1)
 				)
@@
 		(dnp no)
 		(fields_autoplaced yes)
-		(property "Reference" "C2"
+		(property "Reference" "C15"
 			(at 161.29 101.0538 0)
 			(effects
@@
 			)
 		)
-		(property "Footprint" ""
+		(property "Footprint" "Package_TO_SOT_SMD:SOT-23-6_Handsoldering"
 			(at 158.75 102.87 0)
 			(effects
@@
 			(project "PicoBalloon"
 				(path "/0b983980-f4cd-49d3-aecb-9bdb75de805b/ab4eed9b-d1e6-4c70-aac7-9c30168f7593"
-					(reference "C2")
+					(reference "C15")
 					(unit 1)
 				)
@@
 		(dnp no)
 		(fields_autoplaced yes)
-		(property "Reference" "U2"
+		(property "Reference" "U5"
 			(at 120.65 64.77 0)
 			(effects
@@
 			)
 		)
+		(property "LCSC" "https://lcsc.com/product-detail/DC-DC-Converters_MICROCHIP-MCP1640BT-I-CHY_C478087.html"
+			(at 120.65 77.47 0)
+			(effects
+				(font
+					(size 1.27 1.27)
+				)
+				(hide yes)
+			)
+		)
 		(pin "5"
 		)
@@
 			(project "PicoBalloon"
 				(path "/0b983980-f4cd-49d3-aecb-9bdb75de805b/ab4eed9b-d1e6-4c70-aac7-9c30168f7593"
-					(reference "U2")
+					(reference "U5")
 					(unit 1)
 				)
@@
 		(dnp no)
 		(fields_autoplaced yes)
-		(property "Reference" "L1"
+		(property "Reference" "L2"
 			(at 120.65 57.15 90)
 			(effects
@@
 			(project "PicoBalloon"
 				(path "/0b983980-f4cd-49d3-aecb-9bdb75de805b/ab4eed9b-d1e6-4c70-aac7-9c30168f7593"
-					(reference "L1")
+					(reference "L2")
 					(unit 1)
 				)
@@
 		(on_board yes)
 		(dnp no)
-		(property "Reference" "#PWR010"
+		(property "Reference" "#PWR029"
 			(at 158.75 114.3 0)
 			(effects
@@
 			(project "PicoBalloon"
 				(path "/0b983980-f4cd-49d3-aecb-9bdb75de805b/ab4eed9b-d1e6-4c70-aac7-9c30168f7593"
-					(reference "#PWR010")
+					(reference "#PWR029")
 					(unit 1)
 				)
@@
 		(dnp no)
 		(fields_autoplaced yes)
-		(property "Reference" "R11"
+		(property "Reference" "R7"
 			(at 104.14 74.9299 0)
 			(effects
@@
 			(project "PicoBalloon"
 				(path "/0b983980-f4cd-49d3-aecb-9bdb75de805b/ab4eed9b-d1e6-4c70-aac7-9c30168f7593"
-					(reference "R11")
+					(reference "R7")
 					(unit 1)
 				)
@@
 		(dnp no)
 		(fields_autoplaced yes)
-		(property "Reference" "R2"
+		(property "Reference" "R9"
 			(at 142.24 85.0899 0)
 			(effects
@@
 			(project "PicoBalloon"
 				(path "/0b983980-f4cd-49d3-aecb-9bdb75de805b/ab4eed9b-d1e6-4c70-aac7-9c30168f7593"
-					(reference "R2")
+					(reference "R9")
 					(unit 1)
 				)
@@
 		(on_board yes)
 		(dnp no)
-		(property "Reference" "#PWR03"
+		(property "Reference" "#PWR025"
 			(at 87.63 85.09 0)
 			(effects
@@
 			(project "PicoBalloon"
 				(path "/0b983980-f4cd-49d3-aecb-9bdb75de805b/ab4eed9b-d1e6-4c70-aac7-9c30168f7593"
-					(reference "#PWR03")
+					(reference "#PWR025")
 					(unit 1)
 				)
@@
 		(dnp no)
 		(fields_autoplaced yes)
-		(property "Reference" "R1"
+		(property "Reference" "R8"
 			(at 142.24 77.4699 0)
 			(effects
@@
 			(project "PicoBalloon"
 				(path "/0b983980-f4cd-49d3-aecb-9bdb75de805b/ab4eed9b-d1e6-4c70-aac7-9c30168f7593"
-					(reference "R1")
+					(reference "R8")
 					(unit 1)
 				)
@@
 		(dnp no)
 		(fields_autoplaced yes)
-		(property "Reference" "R7"
+		(property "Reference" "R10"
 			(at 161.29 83.8199 0)
 			(effects
@@
 			)
 		)
-		(property "Footprint" "Resistor_SMD:R_0603_1608Metric_Pad0.98x0.95mm_HandSolder"
+		(property "Footprint" "Resistor_SMD:R_2010_5025Metric_Pad1.40x2.65mm_HandSolder"
 			(at 158.75 85.09 0)
 			(effects
@@
 			)
 		)
+		(property "LCSC" "https://lcsc.com/product-detail/image/FRC2010J330-TS_C2907564.html"
+			(at 158.75 85.09 0)
+			(effects
+				(font
+					(size 1.27 1.27)
+				)
+				(hide yes)
+			)
+		)
 		(pin "1"
 		)
@@
 			(project "PicoBalloon"
 				(path "/0b983980-f4cd-49d3-aecb-9bdb75de805b/ab4eed9b-d1e6-4c70-aac7-9c30168f7593"
-					(reference "R7")
+					(reference "R10")
 					(unit 1)
 				)
@@
 		(on_board yes)
 		(dnp no)
-		(property "Reference" "#PWR01"
+		(property "Reference" "#PWR026"
 			(at 120.65 91.44 0)
 			(effects
@@
 			(project "PicoBalloon"
 				(path "/0b983980-f4cd-49d3-aecb-9bdb75de805b/ab4eed9b-d1e6-4c70-aac7-9c30168f7593"
-					(reference "#PWR01")
+					(reference "#PWR026")
 					(unit 1)
 				)
@@
 		(dnp no)
 		(fields_autoplaced yes)
-		(property "Reference" "C1"
+		(property "Reference" "C13"
 			(at 90.17 74.9362 0)
 			(effects
@@
 			(project "PicoBalloon"
 				(path "/0b983980-f4cd-49d3-aecb-9bdb75de805b/ab4eed9b-d1e6-4c70-aac7-9c30168f7593"
-					(reference "C1")
-					(unit 1)
-				)
+					(reference "C13")
+					(unit 1)
+				)

Commit message: Fixed footprints and schematic symbols
Parts:
- C15: footprint Package_TO_SOT_SMD:SOT-23-6_Handsoldering -> Capacitor_THT:CP_Radial_D6.3mm_P2.50mm
Changed lines of the file:
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@@
 			)
 		)
-		(property "Footprint" "Package_TO_SOT_SMD:SOT-23-6_Handsoldering"
+		(property "Footprint" "Capacitor_THT:CP_Radial_D6.3mm_P2.50mm"
 			(at 158.75 102.87 0)
 			(effects
@@
 			)
 		)
-		(property "Datasheet" "~"
+		(property "Datasheet" "https://www.ymin.cn/lithium-ion-capacitor-lic-sla-series-product/"
 			(at 158.75 102.87 0)
 			(effects

Commit message: First PCB layout
Parts:
- C15: footprint Capacitor_THT:CP_Radial_D6.3mm_P2.50mm -> Capacitor_Tantalum_SMD:CP_EIA-3528-12_Kemet-T_HandSolder
Other:
- company: (none) -> Laboratorio Gluon
- title: (none) -> Picoballoon v1
Changed lines of the file:
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@@
 	(generator_version "9.0")
 	(paper "A4")
+	(title_block
+		(title "Picoballoon v1")
+		(date "2025-07-29")
+		(company "Laboratorio Gluon")
+	)
 	(rectangle
 		(start 81.28 63.5)
@@
 				(thickness 0.2032)
 				(bold yes)
+			)
+			(justify left top)
+		)
+	)
+	(text_box "Capacitor data:\n- Max charging current: 100mA\n- Max output current: 150mA"
+		(exclude_from_sim no)
+		(at 168.91 104.14 0)
+		(size 38.1 7.62)
+		(margins 0.9525 0.9525 0.9525 0.9525)
+		(stroke
+			(width 0)
+			(type solid)
+		)
+		(fill
+			(type none)
+		)
+		(effects
+			(font
+				(size 1.27 1.27)
 			)
 			(justify left top)
@@
 			)
 		)
-		(property "Footprint" "Capacitor_THT:CP_Radial_D6.3mm_P2.50mm"
+		(property "Footprint" "Capacitor_Tantalum_SMD:CP_EIA-3528-12_Kemet-T_HandSolder"
 			(at 158.75 102.87 0)
 			(effects

Commit message: Started working on PCB A1.1
Other:
- title: Picoballoon v1 -> Picoballoon A.1.1
Changed lines of the file:
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@@
 	(paper "A4")
 	(title_block
-		(title "Picoballoon v1")
+		(title "Picoballoon A.1.1")
 		(date "2025-07-29")
 		(company "Laboratorio Gluon")
@@
 		(on_board yes)
 		(dnp no)
-		(fields_autoplaced yes)
 		(property "Reference" "C14"
 			(at 152.4 77.4762 0)

Commit message: Updated PCB
Parts:
- C15: value 10F -> 15F
- R10: value 33 -> 16.5
Changed lines of the file:
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@@
 			)
 		)
-		(property "Value" "10F"
+		(property "Value" "15F"
 			(at 161.29 103.5938 0)
 			(effects
@@
 			)
 		)
-		(property "Value" "33"
+		(property "Value" "16.5"
 			(at 161.29 86.3599 0)
 			(effects
