File: Schematics/PicoBalloon/PicoBalloon.kicad_sch (KiCad schematic)
At the start: 31 parts, among them J1 SOLAR_R, J2 SOLAR_L, J3 LORA_ANT, J4 SWD, U1 ATGM336H, U2 AT2659S, U3 TMP235A4DCKR, U4 STM32F103C8Tx

Commit message: Version PCB A1.1
Parts:
- added R12: 33, Resistor_SMD:R_0603_1608Metric_Pad0.98x0.95mm_HandSolder, symbol Device:R_Small
- added R13, R14: 0R, Resistor_SMD:R_0603_1608Metric_Pad0.98x0.95mm_HandSolder, symbol Device:R_Small
- added U7: MT9700, Package_TO_SOT_SMD:SOT-23-5_HandSoldering, symbol gluonLibrary:MT9700
- R3, R4: value 1k -> 3k3
Connections:
- net +3V3: now also U7.5 (Vin); no longer C1.2, C2.2, U1.6 (VBAT), U1.8 (VCC), U2.6 (VDD)
- net GND: now also R12.2, U7.2 (Gnd)
- net GPS_SUPPLY_ENABLE: now reaches U4.13 (PA3)
- net GPS_SUPPLY_ENABLE: now also U7.4 (Enable)
- new net: R12.1, U7.3 (Set)
- new net: C2.2, R14.1, U2.6 (VDD)
- new net: C1.2, R13.1, U1.6 (VBAT), U1.8 (VCC)
- new net SUPPLY_GPS_LNA: R13.2, R14.2, U7.1 (Vout)
- no-connect marks 24 -> 23
Other:
- moved on the sheet: AE1, C1, C10, C11, C12, C2, C3, C4, C5, C8, C9, J1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
